File: joystick_gpio_input/joystick_gpio_input_2p_rasp_part/joystick_gpio_input_2p_rasp_part.kicad_pcb (KiCad board)
At the start: 2 copper layers, 11.8 x 23.3 mm, 3 parts, among them J11 Conn_01x13, J7 Conn_02x09_Odd_Even, J9 Conn_01x13

Commit message: gpio 입력 보드 미세 조정
Signed-off-by: Ju, Gyeong-min <jcmh74@gmail.com>
Routing:
- net /2P_GND: track 33.3 -> 33.9 mm
- net /2P_START: track 12.8 -> 12.3 mm, vias 1 -> 0
Other:
- outline, holes or cut-outs redrawn

Commit message: joystick gpio 스크린샷 추가
Signed-off-by: Ju, Gyeong-min <jcmh74@gmail.com>
Parts:
- renumbered J7 to J1, J9 to J2, J11 to J3
Changed lines of the file:
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@@
   (paper "A4")
   (title_block
-    (title "Raspberry Pie GPIO Input Module")
-    (date "2023-03-26")
+    (title "Raspberry Pie GPIO Input Module (2P Part)")
+    (date "2023-04-02")
     (rev "2")
     (company "Amos Home")
@@
   (net 12 "/2P_TL")
   (net 13 "/2P_TR")
-  (net 14 "unconnected-(J7-Pin_5-Pad5)")
-  (net 15 "unconnected-(J7-Pin_6-Pad6)")
+  (net 14 "unconnected-(J1-Pin_5-Pad5)")
+  (net 15 "unconnected-(J1-Pin_6-Pad6)")
   (footprint "joystick_gpio_input_library:conn_ex_1x13_P1.25mm_Vertical_Right_Labeled" (layer "B.Cu")
     (at 153.7039 92.6576 -90)
@@
     (property "ki_keywords" "connector")
     (attr through_hole)
-    (fp_text reference "J9" (at 7.493 -1.8542 90) (layer "B.SilkS") hide
+    (fp_text reference "J2" (at 7.493 -1.8542 90) (layer "B.SilkS") hide
         (effects (font (size 1 1) (thickness 0.15)) (justify mirror))
     )
@@
     (property "ki_keywords" "connector")
     (attr through_hole)
-    (fp_text reference "J11" (at 7.493 1.8288 90) (layer "B.SilkS") hide
+    (fp_text reference "J3" (at 7.493 1.8288 90) (layer "B.SilkS") hide
         (effects (font (size 1 1) (thickness 0.15)) (justify mirror))
     )
@@
     (property "ki_keywords" "connector")
     (attr through_hole)
-    (fp_text reference "J7" (at -1.27 2.77) (layer "B.SilkS") hide
+    (fp_text reference "J1" (at -1.27 2.77) (layer "B.SilkS") hide
         (effects (font (size 1 1) (thickness 0.15)) (justify mirror))
     )
@@
       (net 10 "/2P_X") (pinfunction "Pin_4") (pintype "passive"))
     (pad "5" thru_hole oval (at 0 -5.08 180) (size 1.7 1.7) (drill 1) (layers "*.Cu" "*.Mask")
-      (net 14 "unconnected-(J7-Pin_5-Pad5)") (pinfunction "Pin_5") (pintype "passive+no_connect"))
+      (net 14 "unconnected-(J1-Pin_5-Pad5)") (pinfunction "Pin_5") (pintype "passive+no_connect"))
     (pad "6" thru_hole oval (at -2.54 -5.08 180) (size 1.7 1.7) (drill 1) (layers "*.Cu" "*.Mask")
-      (net 15 "unconnected-(J7-Pin_6-Pad6)") (pinfunction "Pin_6") (pintype "passive+no_connect"))
+      (net 15 "unconnected-(J1-Pin_6-Pad6)") (pinfunction "Pin_6") (pintype "passive+no_connect"))
     (pad "7" thru_hole oval (at 0 -7.62 180) (size 1.7 1.7) (drill 1) (layers "*.Cu" "*.Mask")
       (net 3 "/2P_DOWN") (pinfunction "Pin_7") (pintype "passive"))
