File: joystick_gpio_input/joystick_gpio_input_main_part/joystick_gpio_input_main_part.kicad_pcb (KiCad board)
At the start: 2 copper layers, 26.2 x 45.3 mm, 22 parts, among them J1 Conn_01x06, J12 Conn_01x15, J2 Conn_01x04, J3 Conn_01x15, J4 Conn_01x15, J5 Conn_01x14

Commit message: gpio 입력 보드 미세 조정
Signed-off-by: Ju, Gyeong-min <jcmh74@gmail.com>
Parts:
- moved J5 0.27 mm to (150.8, 95.1)
Routing:
- net /GND: track 108.1 -> 105.6 mm
- net /C_TL: track 26.4 -> 24.4 mm
- net /SELECT: track 30.2 -> 31.2 mm
- net /C_SELECT: track 12.8 -> 12.0 mm
- net /C_START: track 14.0 -> 13.2 mm
- net /C_A: track 11.4 -> 10.7 mm
Other:
- board size 26.2 x 45.3 mm -> 25.6 x 45.3 mm
- board text added: "*HK"
- board text added: "*R"
- board text added: "*R/*SL/*HK : 1~2:CON, 2~3:GND"
- board text added: "*SL"
- board text added: "G UP DN L *R ST *SL A B X Y TL TR *HK G"
- board text removed: "G UP DN L R* ST SL* A B X Y TL TR HK* G"
- board text removed: "HK*"
- board text removed: "R*"
- board text removed: "R*/SL*/HK* : 1-2:CON, 2-3:GND"
- board text removed: "SL*"

Commit message: joystick gpio 스크린샷 추가
Signed-off-by: Ju, Gyeong-min <jcmh74@gmail.com>
Parts:
- renumbered J12 to J1, J4 to J2, J1 to J4, J2 to J5, J5 to J6
Changed lines of the file:
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@@
     (property "ki_keywords" "connector")
     (attr through_hole)
-    (fp_text reference "J5" (at 8.12 -1.778 90) (layer "F.SilkS") hide
+    (fp_text reference "J6" (at 8.12 -1.778 90) (layer "F.SilkS") hide
         (effects (font (size 1 1) (thickness 0.15)))
     )
@@
     (property "ki_keywords" "connector")
     (attr through_hole)
-    (fp_text reference "J1" (at 7.3152 2.0828 180) (layer "F.SilkS") hide
+    (fp_text reference "J4" (at 7.3152 2.0828 180) (layer "F.SilkS") hide
         (effects (font (size 0.8 0.8) (thickness 0.15)))
     )
@@
     (property "ki_keywords" "connector")
     (attr through_hole)
-    (fp_text reference "J12" (at 0 -2.33) (layer "F.SilkS") hide
+    (fp_text reference "J1" (at 0 -2.33) (layer "F.SilkS") hide
         (effects (font (size 1 1) (thickness 0.15)))
     )
@@
     (property "ki_keywords" "connector")
     (attr through_hole)
-    (fp_text reference "J4" (at 0.0508 -2.032) (layer "F.SilkS") hide
+    (fp_text reference "J2" (at 0.0508 -2.032) (layer "F.SilkS") hide
         (effects (font (size 1 1) (thickness 0.15)))
     )
@@
     (property "ki_keywords" "connector")
     (attr through_hole)
-    (fp_text reference "J2" (at 4.85 2.0828 180) (layer "F.SilkS") hide
-        (effects (font (size 0.8 0.8) (thickness 0.15)))
-    )
+    (fp_text reference "J5" (at 4.85 2.0828 180) (layer "F.SilkS") hide
+        (effects (font (size 0.8 0.8) (thickness 0.15)))
+    )
