File: joystick_gpio_input/joystick_gpio_input_main_part/joystick_gpio_input_main_part.kicad_pcb (KiCad board)
At the start: 2 copper layers, 25.6 x 45.3 mm, 22 parts, among them J1 Conn_01x15, J2 Conn_01x15, J3 Conn_01x15, J4 Conn_01x06, J5 Conn_01x04, J6 Conn_01x14

Commit message: 입력 드라이버 주소 마킹
Signed-off-by: Ju, Gyeong-min <jcmh74@gmail.com>
Other:
- board text added: "https://github.com/amos42/am_joyin"
Changed lines of the file:
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@@
   (gr_circle (center 150.3554 82.3088) (end 151.1554 82.3088)
     (stroke (width 0.1) (type solid)) (fill none) (layer "Edge.Cuts"))
+  (gr_text "https://github.com/amos42/am_joyin" (at 141.6812 117.3734 -90) (layer "B.SilkS")
+    (effects (font (size 1 1) (thickness 0.15)) (justify left bottom mirror))
+  )
   (gr_text "G\nST\nSL\nG" (at 128.5106 119.507) (layer "F.SilkS")
     (effects (font (size 0.8 0.8) (thickness 0.1)) (justify right))
