File: joystick_74hc165_input/joystick_74hc165_input.kicad_pcb (KiCad board)
At the start: 2 copper layers, 53.3 x 39.9 mm, 17 parts, among them J1 Conn_01x18, J2 Conn_02x14_Odd_Even

Commit message: 부품 값 입력
Signed-off-by: Ju, Gyeong-min <jcmh74@gmail.com>
Parts:
- C1: value C -> 22nF
- C2, C3, C4: value C -> 100nF
- RN1, RN4: value R_Network04 -> 10K
- RN2, RN3: value R_Network08 -> 10K
Changed lines of the file:
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@@
     (descr "Through hole straight pin header, 2x14, 2.54mm pitch, double rows")
     (tags "Through hole pin header THT 2x14 2.54mm double row")
-    (property "Sheetfile" "joystick-input.kicad_sch")
+    (property "Sheetfile" "joystick_74hc165_input.kicad_sch")
     (property "Sheetname" "")
     (attr through_hole)
@@
     (descr "Through hole straight pin header, 1x05, 2.54mm pitch, single row")
     (tags "Through hole pin header THT 1x05 2.54mm single row")
-    (property "Sheetfile" "joystick-input.kicad_sch")
+    (property "Sheetfile" "joystick_74hc165_input.kicad_sch")
     (property "Sheetname" "")
     (attr through_hole)
@@
     (descr "Through hole straight pin header, 1x18, 2.54mm pitch, single row")
     (tags "Through hole pin header THT 1x18 2.54mm single row")
-    (property "Sheetfile" "joystick-input.kicad_sch")
+    (property "Sheetfile" "joystick_74hc165_input.kicad_sch")
     (property "Sheetname" "")
     (attr through_hole)
@@
     (descr "16-lead though-hole mounted DIP package, row spacing 7.62 mm (300 mils)")
     (tags "THT DIP DIL PDIP 2.54mm 7.62mm 300mil")
-    (property "Sheetfile" "joystick-input.kicad_sch")
+    (property "Sheetfile" "joystick_74hc165_input.kicad_sch")
     (property "Sheetname" "")
     (attr through_hole)
@@
     (descr "16-lead though-hole mounted DIP package, row spacing 7.62 mm (300 mils)")
     (tags "THT DIP DIL PDIP 2.54mm 7.62mm 300mil")
-    (property "Sheetfile" "joystick-input.kicad_sch")
+    (property "Sheetfile" "joystick_74hc165_input.kicad_sch")
     (property "Sheetname" "")
     (attr through_hole)
@@
     (descr "Capacitor SMD 0805 (2012 Metric), square (rectangular) end terminal, IPC_7351 nominal with elongated pad for handsoldering. (Body size source: IPC-SM-782 page 76, https://www.pcb-3d.com/wordpress/wp-content/uploads/ipc-sm-782a_amendment_1_and_2.pdf, https://docs.google.com/spreadsheets/d/1BsfQQcO9C6DZCsRaXUlFlo91Tg2WpOkGARC1WS5S8t0/edit?usp=sharing), generated with kicad-footprint-generator")
     (tags "capacitor handsolder")
-    (property "Sheetfile" "joystick-input.kicad_sch")
+    (property "Sheetfile" "joystick_74hc165_input.kicad_sch")
     (property "Sheetname" "")
     (attr smd)
@@
       (effects (font (size 0.8 0.8) (thickness 0.15)))
     )
-    (fp_text value "C" (at 0 1.68) (layer "F.Fab")
+    (fp_text value "100nF" (at 0 1.68) (layer "F.Fab")
       (effects (font (size 1 1) (thickness 0.15)))
     )
@@
     (descr "Capacitor SMD 0805 (2012 Metric), square (rectangular) end terminal, IPC_7351 nominal with elongated pad for handsoldering. (Body size source: IPC-SM-782 page 76, https://www.pcb-3d.com/wordpress/wp-content/uploads/ipc-sm-782a_amendment_1_and_2.pdf, https://docs.google.com/spreadsheets/d/1BsfQQcO9C6DZCsRaXUlFlo91Tg2WpOkGARC1WS5S8t0/edit?usp=sharing), generated with kicad-footprint-generator")
     (tags "capacitor handsolder")
-    (property "Sheetfile" "joystick-input.kicad_sch")
+    (property "Sheetfile" "joystick_74hc165_input.kicad_sch")
     (property "Sheetname" "")
     (attr smd)
@@
       (effects (font (size 0.8 0.8) (thickness 0.15)))
     )
-    (fp_text value "C" (at 0 1.68) (layer "F.Fab")
+    (fp_text value "100nF" (at 0 1.68) (layer "F.Fab")
       (effects (font (size 1 1) (thickness 0.15)))
     )
@@
     (descr "5-pin Resistor SIP pack")
     (tags "R")
-    (property "Sheetfile" "joystick-input.kicad_sch")
+    (property "Sheetfile" "joystick_74hc165_input.kicad_sch")
     (property "Sheetname" "")
     (attr through_hole)
@@
       (effects (font (size 0.7 0.8) (thickness 0.15)))
     )
-    (fp_text value "R_Network04" (at 6.35 2.4 90) (layer "F.Fab")
+    (fp_text value "10K" (at 6.35 2.4 90) (layer "F.Fab")
       (effects (font (size 1 1) (thickness 0.15)))
     )
@@
     (descr "5-pin Resistor SIP pack")
     (tags "R")
-    (property "Sheetfile" "joystick-input.kicad_sch")
+    (property "Sheetfile" "joystick_74hc165_input.kicad_sch")
     (property "Sheetname" "")
     (attr through_hole)
@@
       (effects (font (size 0.7 0.8) (thickness 0.15)))
     )
-    (fp_text value "R_Network04" (at 6.35 2.4 90) (layer "F.Fab")
+    (fp_text value "10K" (at 6.35 2.4 90) (layer "F.Fab")
       (effects (font (size 1 1) (thickness 0.15)))
     )
@@
     (descr "9-pin Resistor SIP pack")
     (tags "R")
-    (property "Sheetfile" "joystick-input.kicad_sch")
+    (property "Sheetfile" "joystick_74hc165_input.kicad_sch")
     (property "Sheetname" "")
     (attr through_hole)
@@
       (effects (font (size 0.7 0.8) (thickness 0.15)))
     )
-    (fp_text value "R_Network08" (at 11.43 2.4 90) (layer "F.Fab")
+    (fp_text value "10K" (at 11.43 2.4 90) (layer "F.Fab")
       (effects (font (size 1 1) (thickness 0.15)))
     )
@@
     (descr "16-lead though-hole mounted DIP package, row spacing 7.62 mm (300 mils)")
     (tags "THT DIP DIL PDIP 2.54mm 7.62mm 300mil")
-    (property "Sheetfile" "joystick-input.kicad_sch")
+    (property "Sheetfile" "joystick_74hc165_input.kicad_sch")
     (property "Sheetname" "")
     (attr through_hole)
@@
     (descr "9-pin Resistor SIP pack")
     (tags "R")
-    (property "Sheetfile" "joystick-input.kicad_sch")
+    (property "Sheetfile" "joystick_74hc165_input.kicad_sch")
     (property "Sheetname" "")
     (attr through_hole)
@@
       (effects (font (size 0.7 0.8) (thickness 0.15)))
     )
-    (fp_text value "R_Network08" (at 11.43 2.4 90) (layer "F.Fab")
+    (fp_text value "10K" (at 11.43 2.4 90) (layer "F.Fab")
       (effects (font (size 1 1) (thickness 0.15)))
     )
@@
     (descr "Capacitor SMD 0805 (2012 Metric), square (rectangular) end terminal, IPC_7351 nominal with elongated pad for handsoldering. (Body size source: IPC-SM-782 page 76, https://www.pcb-3d.com/wordpress/wp-content/uploads/ipc-sm-782a_amendment_1_and_2.pdf, https://docs.google.com/spreadsheets/d/1BsfQQcO9C6DZCsRaXUlFlo91Tg2WpOkGARC1WS5S8t0/edit?usp=sharing), generated with kicad-footprint-generator")
     (tags "capacitor handsolder")
-    (property "Sheetfile" "joystick-input.kicad_sch")
+    (property "Sheetfile" "joystick_74hc165_input.kicad_sch")
     (property "Sheetname" "")
     (attr smd)
@@
       (effects (font (size 0.8 0.8) (thickness 0.15)))
     )
-    (fp_text value "C" (at 0 1.68) (layer "F.Fab")
+    (fp_text value "100nF" (at 0 1.68) (layer "F.Fab")
       (effects (font (size 1 1) (thickness 0.15)))
     )
@@
     (descr "Through hole straight pin header, 1x05, 2.54mm pitch, single row")
     (tags "Through hole pin header THT 1x05 2.54mm single row")
-    (property "Sheetfile" "joystick-input.kicad_sch")
+    (property "Sheetfile" "joystick_74hc165_input.kicad_sch")
     (property "Sheetname" "")
     (attr through_hole)
@@
     (descr "SMD Solder Jumper, 1x1.5mm Pads, 0.3mm gap, pads 1-2 bridged with 1 copper strip, labeled with numbers")
     (tags "net tie solder jumper bridged")
-    (property "Sheetfile" "joystick-input.kicad_sch")
+    (property "Sheetfile" "joystick_74hc165_input.kicad_sch")
     (property "Sheetname" "")
     (attr exclude_from_pos_files)
@@
     (descr "SMD Solder Jumper, 1x1.5mm Pads, 0.3mm gap, pads 1-2 bridged with 1 copper strip, labeled with numbers")
     (tags "net tie solder jumper bridged")
-    (property "Sheetfile" "joystick-input.kicad_sch")
+    (property "Sheetfile" "joystick_74hc165_input.kicad_sch")
     (property "Sheetname" "")
     (attr exclude_from_pos_files)
@@
     (descr "Capacitor SMD 0805 (2012 Metric), square (rectangular) end terminal, IPC_7351 nominal with elongated pad for handsoldering. (Body size source: IPC-SM-782 page 76, https://www.pcb-3d.com/wordpress/wp-content/uploads/ipc-sm-782a_amendment_1_and_2.pdf, https://docs.google.com/spreadsheets/d/1BsfQQcO9C6DZCsRaXUlFlo91Tg2WpOkGARC1WS5S8t0/edit?usp=sharing), generated with kicad-footprint-generator")
     (tags "capacitor handsolder")
-    (property "Sheetfile" "joystick-input.kicad_sch")
+    (property "Sheetfile" "joystick_74hc165_input.kicad_sch")
     (property "Sheetname" "")
     (attr smd)
@@
       (effects (font (size 0.8 0.8) (thickness 0.15)))
     )
-    (fp_text value "C" (at 0 1.68) (layer "F.Fab")
-      (effects (font (size 1 1) (thickness 0.15)))
-    )
+    (fp_text value "22nF" (at 0 1.68) (layer "F.Fab")
+      (effects (font (size 1 1) (thickness 0.15)))
+    )

Commit message: 입력 드라이버 주소 마킹
Signed-off-by: Ju, Gyeong-min <jcmh74@gmail.com>
Other:
- board text added: "https://github.com/amos42/am_joyin"
