File: joystick_74hc165_input_1p/joystick_74hc165_input_1p.kicad_pcb (KiCad board)
At the start: 2 copper layers, 53.3 x 29.2 mm, 11 parts, among them J1 Conn_01x18_Male

Commit message: 부품 값 입력
Signed-off-by: Ju, Gyeong-min <jcmh74@gmail.com>
Parts:
- C1, C2: value C -> 100nF
- RN1, RN2: value R_Network08 -> 10K
Changed lines of the file:
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@@
     (descr "Through hole straight pin header, 1x05, 2.54mm pitch, single row")
     (tags "Through hole pin header THT 1x05 2.54mm single row")
-    (property "Sheetfile" "joystick-input.kicad_sch")
+    (property "Sheetfile" "joystick_74hc165_input_1p.kicad_sch")
     (property "Sheetname" "")
     (attr through_hole)
@@
     (descr "16-lead though-hole mounted DIP package, row spacing 7.62 mm (300 mils)")
     (tags "THT DIP DIL PDIP 2.54mm 7.62mm 300mil")
-    (property "Sheetfile" "joystick-input.kicad_sch")
+    (property "Sheetfile" "joystick_74hc165_input_1p.kicad_sch")
     (property "Sheetname" "")
     (attr through_hole)
@@
     (descr "16-lead though-hole mounted DIP package, row spacing 7.62 mm (300 mils)")
     (tags "THT DIP DIL PDIP 2.54mm 7.62mm 300mil")
-    (property "Sheetfile" "joystick-input.kicad_sch")
+    (property "Sheetfile" "joystick_74hc165_input_1p.kicad_sch")
     (property "Sheetname" "")
     (attr through_hole)
@@
     (descr "9-pin Resistor SIP pack")
     (tags "R")
-    (property "Sheetfile" "joystick-input.kicad_sch")
+    (property "Sheetfile" "joystick_74hc165_input_1p.kicad_sch")
     (property "Sheetname" "")
     (attr through_hole)
@@
       (effects (font (size 0.8 0.8) (thickness 0.15)))
     )
-    (fp_text value "R_Network08" (at 11.43 2.4) (layer "F.Fab")
+    (fp_text value "10K" (at 11.43 2.4) (layer "F.Fab")
       (effects (font (size 1 1) (thickness 0.15)))
     )
@@
     (descr "Through hole straight pin header, 1x18, 2.54mm pitch, single row")
     (tags "Through hole pin header THT 1x18 2.54mm single row")
-    (property "Sheetfile" "joystick-input.kicad_sch")
+    (property "Sheetfile" "joystick_74hc165_input_1p.kicad_sch")
     (property "Sheetname" "")
     (attr through_hole)
@@
     (descr "9-pin Resistor SIP pack")
     (tags "R")
-    (property "Sheetfile" "joystick-input.kicad_sch")
+    (property "Sheetfile" "joystick_74hc165_input_1p.kicad_sch")
     (property "Sheetname" "")
     (attr through_hole)
@@
       (effects (font (size 0.8 0.8) (thickness 0.15)))
     )
-    (fp_text value "R_Network08" (at 11.43 2.4) (layer "F.Fab")
+    (fp_text value "10K" (at 11.43 2.4) (layer "F.Fab")
       (effects (font (size 1 1) (thickness 0.15)))
     )
@@
     (descr "Through hole straight pin header, 1x05, 2.54mm pitch, single row")
     (tags "Through hole pin header THT 1x05 2.54mm single row")
-    (property "Sheetfile" "joystick-input.kicad_sch")
+    (property "Sheetfile" "joystick_74hc165_input_1p.kicad_sch")
     (property "Sheetname" "")
     (attr through_hole)
@@
     (descr "C, Disc series, Radial, pin pitch=5.00mm, , diameter*width=4.3*1.9mm^2, Capacitor, http://www.vishay.com/docs/45233/krseries.pdf")
     (tags "C Disc series Radial pin pitch 5.00mm  diameter 4.3mm width 1.9mm Capacitor")
-    (property "Sheetfile" "joystick-input.kicad_sch")
+    (property "Sheetfile" "joystick_74hc165_input_1p.kicad_sch")
     (property "Sheetname" "")
     (attr through_hole)
@@
       (effects (font (size 1 1) (thickness 0.15)))
     )
-    (fp_text value "C" (at 2.5 2.2) (layer "F.Fab")
+    (fp_text value "100nF" (at 2.5 2.2) (layer "F.Fab")
       (effects (font (size 1 1) (thickness 0.15)))
     )
@@
     (descr "C, Disc series, Radial, pin pitch=5.00mm, , diameter*width=4.3*1.9mm^2, Capacitor, http://www.vishay.com/docs/45233/krseries.pdf")
     (tags "C Disc series Radial pin pitch 5.00mm  diameter 4.3mm width 1.9mm Capacitor")
-    (property "Sheetfile" "joystick-input.kicad_sch")
+    (property "Sheetfile" "joystick_74hc165_input_1p.kicad_sch")
     (property "Sheetname" "")
     (attr through_hole)
@@
       (effects (font (size 1 1) (thickness 0.15)))
     )
-    (fp_text value "C" (at 2.5 2.2) (layer "F.Fab")
+    (fp_text value "100nF" (at 2.5 2.2) (layer "F.Fab")
       (effects (font (size 1 1) (thickness 0.15)))
     )
@@
     (descr "SMD Solder Jumper, 1x1.5mm Pads, 0.3mm gap, pads 1-2 bridged with 1 copper strip, labeled with numbers")
     (tags "net tie solder jumper bridged")
-    (property "Sheetfile" "joystick-input.kicad_sch")
+    (property "Sheetfile" "joystick_74hc165_input_1p.kicad_sch")
     (property "Sheetname" "")
     (attr exclude_from_pos_files)
@@
     (descr "SMD Solder Jumper, 1x1.5mm Pads, 0.3mm gap, pads 1-2 bridged with 1 copper strip, labeled with numbers")
     (tags "net tie solder jumper bridged")
-    (property "Sheetfile" "joystick-input.kicad_sch")
+    (property "Sheetfile" "joystick_74hc165_input_1p.kicad_sch")
     (property "Sheetname" "")
     (attr exclude_from_pos_files)

Commit message: 입력 드라이버 주소 마킹
Signed-off-by: Ju, Gyeong-min <jcmh74@gmail.com>
Other:
- board text added: "https://github.com/amos42/am_joyin"
