File: joystick_74hc165_input_jst/joystick_74hc165_input_jst.kicad_pcb (KiCad board)
At the start: 2 copper layers, 71.4 x 38.9 mm, 38 parts, among them J11 Conn_01x05, J12 Conn_01x02, J13 Conn_01x02, J14 Conn_01x02, J15 Conn_01x02, J16 Conn_01x02, J17 Conn_01x02, J18 Conn_01x02, J19 Conn_01x02, J21 Conn_01x05, J22 Conn_01x02, J23 Conn_01x02, J24 Conn_01x02, J25 Conn_01x02, J26 Conn_01x02, J27 Conn_01x02, J28 Conn_01x02, J29 Conn_01x02

Commit message: 부품 값 입력
Signed-off-by: Ju, Gyeong-min <jcmh74@gmail.com>
Parts:
- C1, C2, C3: value C -> 100nF
- RN1, RN2, RN3, RN4, RN5, RN6: value R_Pack04 -> 10K

Commit message: gpio 입력 보드 확장
Signed-off-by: Ju, Gyeong-min <jcmh74@gmail.com>
Other:
- board text added: "Rev.1"
- board text removed: "Rev.3"
Changed lines of the file:
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@@
       (viasonmask false)
       (mode 1)
-      (useauxorigin false)
+      (useauxorigin true)
       (hpglpennumber 1)
       (hpglpenspeed 20)
@@
       (plotinvisibletext false)
       (sketchpadsonfab false)
-      (subtractmaskfromsilk false)
+      (subtractmaskfromsilk true)
       (outputformat 1)
       (mirror false)
@@
   (gr_circle (center 186.5884 79.5528) (end 187.6044 79.5528) (layer "Edge.Cuts") (width 0.15) (fill none))
   (gr_line (start 188.3664 116.6368) (end 116.9924 116.6368) (layer "Edge.Cuts") (width 0.1))
-  (gr_text "Rev.3" (at 125.5014 114.6048) (layer "B.SilkS")
+  (gr_text "Rev.1" (at 125.5014 114.6048) (layer "B.SilkS")
     (effects (font (size 0.7 0.7) (thickness 0.1)) (justify left mirror))
   )

Commit message: 입력 드라이버 주소 마킹
Signed-off-by: Ju, Gyeong-min <jcmh74@gmail.com>
Other:
- board text added: "https://github.com/amos42/am_joyin"
