File: joystick_74hc165_input_smd/joystick_74hc165_input_smd.kicad_pcb (KiCad board)
At the start: 2 copper layers, 53.3 x 29.5 mm, 19 parts, among them J1 Conn_01x18, J2 Conn_02x14_Odd_Even

Commit message: 부품 값 입력
Signed-off-by: Ju, Gyeong-min <jcmh74@gmail.com>
Parts:
- C1, C2, C3: value C -> 100nF
- C4: value C -> 42nF
- RN1, RN2, RN3, RN4, RN5, RN6: value R_Pack04 -> 10K

Commit message: 입력 드라이버 주소 마킹
Signed-off-by: Ju, Gyeong-min <jcmh74@gmail.com>
Other:
- board text added: "https://github.com/amos42/am_joyin"
